File: accel-chain.brd (EAGLE design)
At the start: 25.1 x 18.3 mm, 15 parts, among them IC1 ADXL330, IC2 ATTINY87/167AUTOMOTIVE, U1 ISL3179EIBZ

Commit message: Now with picoblade connectors
Parts:
- removed ISP1: AVRISP-6, adafruit:AVRISP
- added U$2: PICOBLADE-6-MOLEX_53261-0671, glacsweb:PICOBLADE_6-MOLEX_53261-0671
- moved C1 6.65 mm to (22.5, 16.4), turned to 0 degrees
- moved C6 4.33 mm to (19.6, 13.6)
- moved C5 2.62 mm to (18.3, 14.5), turned to 0 degrees
- moved C4 2.44 mm to (13.3, 14.5), turned to 180 degrees
Connections:
- net !RESET: now also U$2.5; no longer ISP1.5
- net GND: now also U$2.6; no longer ISP1.6
- net MISO: now also U$2.1; no longer ISP1.1
- net MOSI: now also U$2.4; no longer ISP1.4
- net SCK: now also U$2.3; no longer ISP1.3
- net VCC: now also U$2.2; no longer ISP1.2
- net X: now also IC2.15; no longer IC2.3
Routing:
- net X: track 18.0 -> 42.5 mm, vias 0 -> 2
- net GND: track 46.0 -> 68.2 mm, vias 1 -> 7
- net VCC: track 51.3 -> 35.9 mm, vias 0 -> 1
- net SCK: track 9.05 -> 16.3 mm
- net MOSI: track 5.55 -> 12.2 mm
- net !RESET: track 15.8 -> 20.1 mm, vias 2 -> 3
- net MISO: track 10.6 -> 8.35 mm, vias 2 -> 0
- net Z: track 19.4 -> 21.3 mm
- net Y: track 25.6 -> 27.3 mm
- net 3V3: track 17.4 -> 18.1 mm, vias 4 -> 6
Other:
- board size 25.1 x 18.3 mm -> 25.1 x 16.5 mm
