File: temp-accel-chain.brd (EAGLE design)
At the start: 29.2 x 10.5 mm, 10 parts, among them U1 ADT7420UCPZ-R2, U2 ADXL345

Commit message: removed unneeded resistor on add select pins
Parts:
- removed R1: 10K, resistor:R0603
Connections:
- removed net ADD_SEL: JP1.2, R1.1
- net ADD: now also JP1.2; no longer R1.2
Routing:
- net ADD_SEL: track 14.6 -> 0.00 mm
- net ADD: track 21.6 -> 31.7 mm
Changed lines of the file:
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@@
 <setting verticaltext="up"/>
 </settings>
-<grid distance="5" unitdist="mil" unit="mm" style="lines" multiple="1" display="no" altdistance="1" altunitdist="mil" altunit="mil"/>
+<grid distance="5" unitdist="mil" unit="mil" style="lines" multiple="1" display="no" altdistance="1" altunitdist="mil" altunit="mil"/>
 <layers>
 <layer number="1" name="Top" color="4" fill="1" visible="yes" active="yes"/>
@@
 <attribute name="VALUE" x="17.78" y="4.9799" size="0.02" layer="27" rot="R90"/>
 </element>
-<element name="R1" library="resistor" package="R0603" value="10K" x="8.636" y="4.318" smashed="yes" rot="R90"/>
 <element name="U2" library="SparkFun-Sensors" package="LGA14" value="ADXL345" x="15.113" y="4.953" smashed="yes" rot="MR270"/>
 <element name="C2" library="resistor" package="C0805" value="" x="29.972" y="2.54" smashed="yes" rot="R270">
@@
 </signal>
 <signal name="ADD">
-<contactref element="R1" pad="2"/>
 <contactref element="U1" pad="4"/>
 <contactref element="U1" pad="3"/>
 <wire x1="10.7188" y1="4.1148" x2="10.7188" y2="4.7498" width="0.254" layer="1"/>
-<wire x1="8.636" y1="5.168" x2="9.1576" y2="5.168" width="0.254" layer="1"/>
-<wire x1="9.1576" y1="5.168" x2="9.5758" y2="4.7498" width="0.254" layer="1"/>
-<wire x1="9.5758" y1="4.7498" x2="10.7188" y2="4.7498" width="0.254" layer="1"/>
 <contactref element="U2" pad="12"/>
 <wire x1="16.213" y1="3.753" x2="17.088" y2="3.753" width="0.254" layer="16"/>
@@
 <wire x1="11.049" y1="3.048" x2="10.7188" y2="3.3782" width="0.254" layer="1"/>
 <wire x1="10.7188" y1="3.3782" x2="10.7188" y2="4.1148" width="0.254" layer="1"/>
-</signal>
-<signal name="ADD_SEL">
-<contactref element="R1" pad="1"/>
 <contactref element="JP1" pad="2"/>
 <wire x1="17.78" y1="5.08" x2="18.923" y2="5.08" width="0.254" layer="1"/>
-<wire x1="10.922" y1="2.286" x2="18.542" y2="2.286" width="0.254" layer="1"/>
 <wire x1="18.542" y1="2.286" x2="19.05" y2="2.794" width="0.254" layer="1"/>
 <wire x1="19.05" y1="2.794" x2="19.05" y2="4.953" width="0.254" layer="1"/>
 <wire x1="19.05" y1="4.953" x2="18.923" y2="5.08" width="0.254" layer="1"/>
-<wire x1="8.636" y1="3.468" x2="9.74" y2="3.468" width="0.254" layer="1"/>
-<wire x1="9.74" y1="3.468" x2="10.922" y2="2.286" width="0.254" layer="1"/>
+<wire x1="18.542" y1="2.286" x2="11.176" y2="2.286" width="0.3048" layer="1"/>
+<wire x1="11.176" y1="2.286" x2="11.049" y2="2.413" width="0.3048" layer="1"/>
+<wire x1="11.049" y1="2.413" x2="11.049" y2="3.048" width="0.3048" layer="1"/>
 </signal>
 </signals>
