File: interface.brd (EAGLE design)
At the start: 36.3 x 29.1 mm, 25 parts, among them U1 ISL3179EIBZ, U2 ATMEGA328P

Commit message: track lengths now within 0.2% for rs485
Connections:
- net AY renamed 485_P
- net BZ renamed 485_N
Routing:
- net 485_P: track 53.8 -> 50.4 mm
- net 485_N: track 53.8 -> 50.8 mm, vias 1 -> 2
Changed lines of the file:
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@@
 <?xml version="1.0" encoding="utf-8"?>
 <!DOCTYPE eagle SYSTEM "eagle.dtd">
-<eagle version="6.5.0">
+<eagle version="6.6.0">
 <drawing>
 <settings>
@@
 <setting verticaltext="up"/>
 </settings>
-<grid distance="5" unitdist="mil" unit="mm" style="lines" multiple="1" display="yes" altdistance="1" altunitdist="mil" altunit="mil"/>
+<grid distance="5" unitdist="mil" unit="mil" style="lines" multiple="1" display="yes" altdistance="1" altunitdist="mil" altunit="mil"/>
 <layers>
 <layer number="1" name="Top" color="4" fill="1" visible="yes" active="yes"/>
@@
 <classes>
 <class number="0" name="default" width="0" drill="0">
+</class>
+<class number="1" name="rs485" width="0.3048" drill="0">
+<clearance class="1" value="0.1524"/>
 </class>
 </classes>
@@
 <wire x1="-31.965" y1="17.526" x2="-30.822" y2="16.383" width="0.3048" layer="1"/>
 </signal>
-<signal name="AY">
-<contactref element="U1" pad="6"/>
-<contactref element="JP2" pad="2"/>
-<contactref element="JP1" pad="2"/>
-<wire x1="-35.687" y1="14.224" x2="-33.782" y2="14.224" width="0.6096" layer="16"/>
-<wire x1="-33.782" y1="14.224" x2="-32.512" y2="12.954" width="0.6096" layer="16"/>
-<wire x1="-32.512" y1="12.954" x2="-32.512" y2="8.128" width="0.6096" layer="16"/>
-<wire x1="-32.512" y1="8.128" x2="-31.75" y2="7.366" width="0.6096" layer="16"/>
-<wire x1="-31.75" y1="7.366" x2="-16.256" y2="7.366" width="0.6096" layer="16"/>
-<via x="-16.256" y="7.366" extent="1-16" drill="0.4826"/>
-<wire x1="-16.256" y1="7.366" x2="-8.382" y2="7.366" width="0.6096" layer="1"/>
-<via x="-8.382" y="7.366" extent="1-16" drill="0.4826"/>
-<wire x1="-8.382" y1="7.366" x2="-6.223" y2="7.366" width="0.6096" layer="16"/>
-<wire x1="-6.223" y1="7.366" x2="-5.588" y2="8.001" width="0.6096" layer="16"/>
-<wire x1="-5.588" y1="8.001" x2="-5.588" y2="13.208" width="0.6096" layer="16"/>
-<wire x1="-5.588" y1="13.208" x2="-7.112" y2="14.732" width="0.6096" layer="16"/>
-<wire x1="-7.112" y1="14.732" x2="-8.255" y2="14.732" width="0.6096" layer="16"/>
-<wire x1="-8.255" y1="14.732" x2="-7.874" y2="14.986" width="0.6096" layer="16"/>
-<wire x1="-16.256" y1="7.366" x2="-16.256" y2="8.128" width="0.3048" layer="16"/>
-<wire x1="-16.256" y1="8.128" x2="-17.526" y2="9.398" width="0.3048" layer="16"/>
-<wire x1="-17.526" y1="9.398" x2="-18.415" y2="9.398" width="0.3048" layer="16"/>
-<wire x1="-18.415" y1="9.398" x2="-19.177" y2="10.16" width="0.3048" layer="16"/>
-<wire x1="-19.177" y1="10.16" x2="-19.177" y2="12.573" width="0.3048" layer="16"/>
-<wire x1="-19.177" y1="12.573" x2="-19.812" y2="13.208" width="0.3048" layer="16"/>
-<wire x1="-19.812" y1="13.208" x2="-20.7518" y2="13.208" width="0.3048" layer="16"/>
-</signal>
-<signal name="BZ">
+<signal name="485_N" class="1">
 <contactref element="U1" pad="7"/>
 <contactref element="JP1" pad="3"/>
 <contactref element="JP2" pad="3"/>
-<wire x1="-35.687" y1="11.684" x2="-34.417" y2="11.684" width="0.6096" layer="16"/>
-<wire x1="-34.417" y1="11.684" x2="-33.528" y2="10.795" width="0.6096" layer="16"/>
-<wire x1="-33.528" y1="10.795" x2="-33.528" y2="7.493" width="0.6096" layer="16"/>
-<wire x1="-33.528" y1="7.493" x2="-32.258" y2="6.223" width="0.6096" layer="16"/>
-<wire x1="-32.258" y1="6.223" x2="-14.605" y2="6.223" width="0.6096" layer="16"/>
-<via x="-14.605" y="6.223" extent="1-16" drill="0.4826"/>
-<wire x1="-14.605" y1="6.223" x2="-6.604" y2="6.223" width="0.6096" layer="1"/>
-<wire x1="-6.604" y1="6.223" x2="-5.461" y2="7.366" width="0.6096" layer="1"/>
-<wire x1="-5.461" y1="7.366" x2="-5.461" y2="11.811" width="0.6096" layer="1"/>
-<wire x1="-5.461" y1="11.811" x2="-5.969" y2="12.319" width="0.6096" layer="1"/>
-<wire x1="-5.969" y1="12.319" x2="-7.874" y2="12.446" width="0.6096" layer="1"/>
-<wire x1="-14.605" y1="6.223" x2="-14.605" y2="7.493" width="0.3048" layer="16"/>
-<wire x1="-14.605" y1="7.493" x2="-17.526" y2="10.414" width="0.3048" layer="16"/>
-<wire x1="-17.526" y1="10.414" x2="-18.288" y2="10.414" width="0.3048" layer="16"/>
-<wire x1="-18.288" y1="10.414" x2="-18.669" y2="10.795" width="0.3048" layer="16"/>
-<wire x1="-18.669" y1="10.795" x2="-18.669" y2="13.335" width="0.3048" layer="16"/>
-<wire x1="-18.669" y1="13.335" x2="-19.812" y2="14.478" width="0.3048" layer="16"/>
-<wire x1="-19.812" y1="14.478" x2="-20.7518" y2="14.478" width="0.3048" layer="16"/>
+<wire x1="-35.687" y1="11.684" x2="-34.7726" y2="12.5984" width="0.3048" layer="16"/>
+<wire x1="-34.7726" y1="12.5984" x2="-33.62269375" y2="12.5984" width="0.3048" layer="16"/>
+<wire x1="-33.62269375" y1="12.5984" x2="-32.7406" y2="11.71630625" width="0.3048" layer="16"/>
+<wire x1="-32.7406" y1="11.71630625" x2="-32.7406" y2="7.52530625" width="0.3048" layer="16"/>
+<wire x1="-32.7406" y1="7.52530625" x2="-31.46369375" y2="6.2484" width="0.3048" layer="16"/>
+<wire x1="-31.46369375" y1="6.2484" x2="-16.383" y2="6.2484" width="0.3048" layer="16"/>
+<via x="-16.383" y="6.0984" extent="1-16" drill="0.3" shape="square"/>
+<wire x1="-16.383" y1="6.2484" x2="-16.383" y2="6.0984" width="0.3048" layer="1"/>
+<wire x1="-16.383" y1="6.2484" x2="-16.383" y2="6.0984" width="0.3048" layer="16"/>
+<wire x1="-10.82730625" y1="6.2484" x2="-16.383" y2="6.2484" width="0.3048" layer="1"/>
+<wire x1="-10.82730625" y1="6.2484" x2="-9.6774" y2="7.39830625" width="0.3048" layer="1"/>
+<wire x1="-9.6774" y1="7.39830625" x2="-9.6774" y2="8.382" width="0.3048" layer="1"/>
+<via x="-9.5274" y="8.382" extent="1-16" drill="0.3" shape="square"/>
+<wire x1="-9.6774" y1="8.382" x2="-9.5274" y2="8.382" width="0.3048" layer="16"/>
+<wire x1="-9.6774" y1="8.382" x2="-9.5274" y2="8.382" width="0.3048" layer="1"/>
+<wire x1="-7.874" y1="12.446" x2="-8.1534" y2="12.446" width="0.3048" layer="16"/>
+<wire x1="-9.6774" y1="8.382" x2="-9.6774" y2="8.7884" width="0.3048" layer="16"/>
+<wire x1="-9.6774" y1="8.7884" x2="-9.779" y2="9.017" width="0.3048" layer="16"/>
+<wire x1="-9.779" y1="9.017" x2="-9.779" y2="12.319" width="0.3048" layer="16"/>
+<wire x1="-9.779" y1="12.319" x2="-9.652" y2="12.446" width="0.3048" layer="16"/>
+<wire x1="-9.652" y1="12.446" x2="-7.874" y2="12.446" width="0.3048" layer="16"/>
+<wire x1="-20.7518" y1="14.478" x2="-19.74270625" y2="14.478" width="0.3048" layer="16"/>
+<wire x1="-19.74270625" y1="14.478" x2="-18.5674" y2="13.30269375" width="0.3048" layer="16"/>
+<wire x1="-18.5674" y1="10.63569375" x2="-18.5674" y2="13.30269375" width="0.3048" layer="16"/>
+<wire x1="-18.5674" y1="10.63569375" x2="-17.81230625" y2="9.8806" width="0.3048" layer="16"/>
+<wire x1="-17.81230625" y1="9.8806" x2="-17.399" y2="9.8806" width="0.3048" layer="16"/>
+<wire x1="-17.399" y1="9.8806" x2="-16.383" y2="8.8646" width="0.3048" layer="16"/>
+<wire x1="-16.383" y1="8.8646" x2="-16.383" y2="6.0984" width="0.3048" layer="16"/>
 </signal>
 <signal name="RX">
@@
 <wire x1="-14.859" y1="23.876" x2="-14.859" y2="23.114" width="0.3048" layer="16"/>
 </signal>
+<signal name="485_P" class="1">
+<contactref element="U1" pad="6"/>
+<contactref element="JP2" pad="2"/>
+<contactref element="JP1" pad="2"/>
+<wire x1="-35.687" y1="14.224" x2="-34.5186" y2="13.0556" width="0.3048" layer="16"/>
+<wire x1="-34.5186" y1="13.0556" x2="-33.43330625" y2="13.0556" width="0.3048" layer="16"/>
+<wire x1="-33.43330625" y1="13.0556" x2="-32.2834" y2="11.90569375" width="0.3048" layer="16"/>
+<wire x1="-32.2834" y1="11.90569375" x2="-32.2834" y2="7.71469375" width="0.3048" layer="16"/>
+<wire x1="-32.2834" y1="7.71469375" x2="-31.27430625" y2="6.7056" width="0.3048" layer="16"/>
+<wire x1="-31.27430625" y1="6.7056" x2="-17.272" y2="6.7056" width="0.3048" layer="16"/>
+<via x="-17.272" y="6.8556" extent="1-16" drill="0.3" shape="square"/>
+<wire x1="-17.272" y1="6.7056" x2="-17.272" y2="6.8556" width="0.3048" layer="1"/>
+<wire x1="-17.272" y1="6.7056" x2="-17.272" y2="6.8556" width="0.3048" layer="16"/>
+<wire x1="-11.01669375" y1="6.7056" x2="-17.272" y2="6.7056" width="0.3048" layer="1"/>
+<wire x1="-11.01669375" y1="6.7056" x2="-10.1346" y2="7.58769375" width="0.3048" layer="1"/>
+<wire x1="-10.1346" y1="7.58769375" x2="-10.1346" y2="8.382" width="0.3048" layer="1"/>
+<via x="-10.2846" y="8.382" extent="1-16" drill="0.3" shape="square"/>
+<wire x1="-10.4394" y1="8.382" x2="-10.2846" y2="8.382" width="0.3048" layer="16"/>
+<wire x1="-10.1346" y1="8.382" x2="-10.2846" y2="8.382" width="0.3048" layer="1"/>
+<wire x1="-7.874" y1="14.986" x2="-9.271" y2="14.986" width="0.3048" layer="16"/>
+<wire x1="-9.271" y1="14.986" x2="-10.287" y2="13.97" width="0.3048" layer="16"/>
+<wire x1="-10.287" y1="13.97" x2="-10.287" y2="8.3844" width="0.3048" layer="16"/>
+<wire x1="-10.287" y1="8.3844" x2="-10.2846" y2="8.382" width="0.3048" layer="16"/>
+<wire x1="-20.7518" y1="13.208" x2="-19.0246" y2="13.208" width="0.3048" layer="16"/>
+<wire x1="-19.0246" y1="10.44630625" x2="-19.0246" y2="13.208" width="0.3048" layer="16"/>
+<wire x1="-19.0246" y1="10.44630625" x2="-18.00169375" y2="9.4234" width="0.3048" layer="16"/>
+<wire x1="-18.00169375" y1="9.4234" x2="-17.526" y2="9.4234" width="0.3048" layer="16"/>
+<wire x1="-17.526" y1="9.4234" x2="-17.272" y2="9.1694" width="0.3048" layer="16"/>
+<wire x1="-17.272" y1="9.1694" x2="-17.272" y2="6.8556" width="0.3048" layer="16"/>
+</signal>
 </signals>
